File: KiCad/videopac-usbcart-kicad5.kicad_pcb (KiCad board)
At the start: 2 copper layers, 63 x 85 mm, 27 parts, among them J1 Videopac-edgeconnector, J2 USB_B, J3 AVR-ISP-10, J4 Conn_01x01_Male, U1 ATmega16A-AU, U2 IDT7006PF-PN64, Y1 12MHz

Commit message: rev 1.1
Routing:
- net /5V_CART: track 40.4 -> 50.3 mm, vias 1 -> 3
- net /A0: track 28.8 -> 33.4 mm
- net /#PSEN: track 26.6 -> 22.7 mm
- net /A3: track 31.5 -> 28.1 mm
- net /A4: track 24.1 -> 26.1 mm
- net /A1: track 28.9 -> 30.4 mm
- net /A2: track 29.7 -> 28.9 mm
Other:
- outline, holes or cut-outs redrawn
- rule pad_to_mask_clearance: 0.051 -> 0.0508
- board text added: "Videopac USBCART 1.1"
- board text removed: "Videopac USBCART 1.0beta"
